Commit message: chg: restructure the urdf files

File: franka_description/robots/mixed/mixed_dual_panda_arm.urdf.xacro (robot description, xacro)
@@ -6,5 +6,4 @@
   <xacro:arg name="hand_2" default="false"/> <!-- Should a franka_gripper be mounted at the flange?" -->
   <xacro:arg name="robot_ip_1" default=""/> <!-- IP address or hostname of the robot" -->
-  <xacro:arg name="robot_ip_2" default=""/> <!-- IP address or hostname of the robot" -->
   <xacro:arg name="use_fake_hardware" default="false"/>
   <xacro:arg name="fake_sensor_commands" default="false"/>
@@ -23,5 +22,5 @@
     </collision>
   </link>
-  <xacro:include filename="$(find franka_description)/robots/panda_arm.xacro"/>
+  <xacro:include filename="$(find franka_description)/robots/common/panda_arm.xacro"/>
   <!--
   <xacro:panda_arm arm_id="$(arg arm_id_1)" connected_to="base_link" rpy="${-90 * pi/180} 0 ${-90 * pi/180}"  xyz="-143.26e-3 +600e-3 924.51e-3" safety_distance="0.03"/>
@@ -31,12 +30,14 @@
   <xacro:panda_arm arm_id="$(arg arm_id_2)" connected_to="base_link" rpy="0 0 0"  xyz="0 -0.26 0" safety_distance="0.03"/>
   <xacro:if value="$(arg hand_1)">
-    <xacro:include filename="$(find franka_description)/robots/hand.xacro"/>
+    <xacro:include filename="$(find franka_description)/robots/common/hand.xacro"/>
     <xacro:hand ns="$(arg arm_id_1)" rpy="0 0 ${-pi/4}" connected_to="$(arg arm_id_1)_link8" safety_distance="0.03"/>
   </xacro:if>
   <xacro:if value="$(arg hand_2)">
-    <xacro:include filename="$(find franka_description)/robots/hand.xacro"/>
+    <xacro:include filename="$(find franka_description)/robots/common/hand.xacro"/>
     <xacro:hand ns="$(arg arm_id_2)" rpy="0 0 ${-pi/4}" connected_to="$(arg arm_id_2)_link8" safety_distance="0.03"/>
   </xacro:if>
-  <xacro:include filename="$(find franka_description)/robots/dual_panda_arm.ros2_control.xacro"/>
-  <xacro:panda_arm_ros2_control ns_1="$(arg arm_id_1)" ns_2="$(arg arm_id_2)" robot_ip_1="$(arg robot_ip_1)" robot_ip_2="$(arg robot_ip_2)" use_fake_hardware="$(arg use_fake_hardware)" fake_sensor_commands="$(arg fake_sensor_commands)"/>
+  <xacro:include filename="$(find franka_description)/robots/real/panda_arm.ros2_control.xacro"/>
+  <xacro:panda_arm_ros2_control ns="$(arg arm_id_1)" robot_ip="$(arg robot_ip_1)" use_fake_hardware="$(arg use_fake_hardware)" fake_sensor_commands="$(arg fake_sensor_commands)"/>
+  <xacro:include filename="$(find franka_description)/robots/sim/panda_arm_sim.ros2_control.xacro"/>
+  <xacro:panda_arm_sim_ros2_control ns="$(arg arm_id_2)" hand="$(arg hand_2)"/>
 </robot>

File: franka_description/robots/mixed/mixed_quad_panda_arm.urdf.xacro (robot description, xacro)
@@ -11,6 +11,4 @@
   <xacro:arg name="robot_ip_1" default=""/> <!-- IP address or hostname of the robot" -->
   <xacro:arg name="robot_ip_2" default=""/> <!-- IP address or hostname of the robot" -->
-  <xacro:arg name="scene_xml" default=""/>
-  <xacro:arg name="mj_yaml" default=""/>
   <xacro:arg name="use_fake_hardware" default="false"/>
   <xacro:arg name="fake_sensor_commands" default="false"/>
@@ -29,5 +27,5 @@
     </collision>
   </link>
-  <xacro:include filename="$(find franka_description)/robots/panda_arm.xacro"/>
+  <xacro:include filename="$(find franka_description)/robots/common/panda_arm.xacro"/>
   <xacro:panda_arm arm_id="$(arg arm_id_1)" connected_to="base_link" rpy="0 0 0"  xyz="-0.4 +0.26 0" safety_distance="0.03"/>
   <xacro:panda_arm arm_id="$(arg arm_id_2)" connected_to="base_link" rpy="0 0 0"  xyz="-0.4 -0.26 0" safety_distance="0.03"/>
@@ -35,22 +33,22 @@
   <xacro:panda_arm arm_id="$(arg arm_id_2)" connected_to="base_link" rpy="0 0 0"  xyz="+0.4 -0.26 0" safety_distance="0.03"/>
   <xacro:if value="$(arg hand_1)">
-    <xacro:include filename="$(find franka_description)/robots/hand.xacro"/>
+    <xacro:include filename="$(find franka_description)/robots/common/hand.xacro"/>
     <xacro:hand ns="$(arg arm_id_1)" rpy="0 0 ${-pi/4}" connected_to="$(arg arm_id_1)_link8" safety_distance="0.03"/>
   </xacro:if>
   <xacro:if value="$(arg hand_2)">
-    <xacro:include filename="$(find franka_description)/robots/hand.xacro"/>
+    <xacro:include filename="$(find franka_description)/robots/common/hand.xacro"/>
     <xacro:hand ns="$(arg arm_id_2)" rpy="0 0 ${-pi/4}" connected_to="$(arg arm_id_2)_link8" safety_distance="0.03"/>
   </xacro:if>
   <xacro:if value="$(arg hand_3)">
-    <xacro:include filename="$(find franka_description)/robots/hand.xacro"/>
+    <xacro:include filename="$(find franka_description)/robots/common/hand.xacro"/>
     <xacro:hand ns="$(arg arm_id_3)" rpy="0 0 ${-pi/4}" connected_to="$(arg arm_id_3)_link8" safety_distance="0.03"/>
   </xacro:if>
   <xacro:if value="$(arg hand_4)">
-    <xacro:include filename="$(find franka_description)/robots/hand.xacro"/>
+    <xacro:include filename="$(find franka_description)/robots/common/hand.xacro"/>
     <xacro:hand ns="$(arg arm_id_4)" rpy="0 0 ${-pi/4}" connected_to="$(arg arm_id_4)_link8" safety_distance="0.03"/>
   </xacro:if>
-  <xacro:include filename="$(find franka_description)/robots/dual_panda_arm.ros2_control.xacro"/>
+  <xacro:include filename="$(find franka_description)/robots/real/dual_panda_arm.ros2_control.xacro"/>
   <xacro:panda_arm_ros2_control ns_1="$(arg arm_id_1)" ns_2="$(arg arm_id_2)" robot_ip_1="$(arg robot_ip_1)" robot_ip_2="$(arg robot_ip_2)" use_fake_hardware="$(arg use_fake_hardware)" fake_sensor_commands="$(arg fake_sensor_commands)"/>
-  <xacro:include filename="$(find franka_description)/robots/dual_panda_arm_sim.ros2_control.xacro"/>
-  <xacro:panda_arm_sim_ros2_control ns_1="$(arg arm_id_3)" ns_2="$(arg arm_id_4)" hand_1="$(arg hand_3)" hand_2="$(arg hand_4)" scene_xml="$(arg scene_xml)" mj_yaml="$(arg mj_yaml)"/>
+  <xacro:include filename="$(find franka_description)/robots/sim/dual_panda_arm_sim.ros2_control.xacro"/>
+  <xacro:panda_arm_sim_ros2_control ns_1="$(arg arm_id_3)" ns_2="$(arg arm_id_4)" hand_1="$(arg hand_3)" hand_2="$(arg hand_4)"/>
 </robot>

File: franka_description/robots/real/dual_panda_arm.urdf.xacro (robot description, xacro)
@@ -6,6 +6,5 @@
   <xacro:arg name="hand_2" default="false"/> <!-- Should a franka_gripper be mounted at the flange?" -->
   <xacro:arg name="robot_ip_1" default=""/> <!-- IP address or hostname of the robot" -->
-  <xacro:arg name="scene_xml" default=""/>
-  <xacro:arg name="mj_yaml" default=""/>
+  <xacro:arg name="robot_ip_2" default=""/> <!-- IP address or hostname of the robot" -->
   <xacro:arg name="use_fake_hardware" default="false"/>
   <xacro:arg name="fake_sensor_commands" default="false"/>
@@ -24,5 +23,5 @@
     </collision>
   </link>
-  <xacro:include filename="$(find franka_description)/robots/panda_arm.xacro"/>
+  <xacro:include filename="$(find franka_description)/robots/common/panda_arm.xacro"/>
   <!--
   <xacro:panda_arm arm_id="$(arg arm_id_1)" connected_to="base_link" rpy="${-90 * pi/180} 0 ${-90 * pi/180}"  xyz="-143.26e-3 +600e-3 924.51e-3" safety_distance="0.03"/>
@@ -32,14 +31,12 @@
   <xacro:panda_arm arm_id="$(arg arm_id_2)" connected_to="base_link" rpy="0 0 0"  xyz="0 -0.26 0" safety_distance="0.03"/>
   <xacro:if value="$(arg hand_1)">
-    <xacro:include filename="$(find franka_description)/robots/hand.xacro"/>
+    <xacro:include filename="$(find franka_description)/robots/common/hand.xacro"/>
     <xacro:hand ns="$(arg arm_id_1)" rpy="0 0 ${-pi/4}" connected_to="$(arg arm_id_1)_link8" safety_distance="0.03"/>
   </xacro:if>
   <xacro:if value="$(arg hand_2)">
-    <xacro:include filename="$(find franka_description)/robots/hand.xacro"/>
+    <xacro:include filename="$(find franka_description)/robots/common/hand.xacro"/>
     <xacro:hand ns="$(arg arm_id_2)" rpy="0 0 ${-pi/4}" connected_to="$(arg arm_id_2)_link8" safety_distance="0.03"/>
   </xacro:if>
-  <xacro:include filename="$(find franka_description)/robots/panda_arm.ros2_control.xacro"/>
-  <xacro:panda_arm_ros2_control ns="$(arg arm_id_1)" robot_ip="$(arg robot_ip_1)" use_fake_hardware="$(arg use_fake_hardware)" fake_sensor_commands="$(arg fake_sensor_commands)"/>
-  <xacro:include filename="$(find franka_description)/robots/panda_arm_sim.ros2_control.xacro"/>
-  <xacro:panda_arm_sim_ros2_control ns="$(arg arm_id_2)" hand="$(arg hand_2)" scene_xml="$(arg scene_xml)" mj_yaml="$(arg mj_yaml)"/>
+  <xacro:include filename="$(find franka_description)/robots/real/dual_panda_arm.ros2_control.xacro"/>
+  <xacro:panda_arm_ros2_control ns_1="$(arg arm_id_1)" ns_2="$(arg arm_id_2)" robot_ip_1="$(arg robot_ip_1)" robot_ip_2="$(arg robot_ip_2)" use_fake_hardware="$(arg use_fake_hardware)" fake_sensor_commands="$(arg fake_sensor_commands)"/>
 </robot>

File: franka_description/robots/real/panda_arm.urdf.xacro (robot description, xacro)
@@ -6,11 +6,11 @@
   <xacro:arg name="use_fake_hardware" default="false"/>
   <xacro:arg name="fake_sensor_commands" default="false"/>
-  <xacro:include filename="$(find franka_description)/robots/panda_arm.xacro"/>
+  <xacro:include filename="$(find franka_description)/robots/common/panda_arm.xacro"/>
   <xacro:panda_arm arm_id="$(arg arm_id)" safety_distance="0.03"/>
   <xacro:if value="$(arg hand)">
-    <xacro:include filename="$(find franka_description)/robots/hand.xacro"/>
+    <xacro:include filename="$(find franka_description)/robots/common/hand.xacro"/>
     <xacro:hand ns="$(arg arm_id)" rpy="0 0 ${-pi/4}" connected_to="$(arg arm_id)_link8" safety_distance="0.03"/>
   </xacro:if>
-  <xacro:include filename="$(find franka_description)/robots/panda_arm.ros2_control.xacro"/>
+  <xacro:include filename="$(find franka_description)/robots/real/panda_arm.ros2_control.xacro"/>
   <xacro:panda_arm_ros2_control ns="$(arg arm_id)" robot_ip="$(arg robot_ip)" use_fake_hardware="$(arg use_fake_hardware)" fake_sensor_commands="$(arg fake_sensor_commands)"/>
 </robot>

File: franka_description/robots/sim/dual_panda_arm_sim.ros2_control.xacro (robot description, xacro)
@@ -1,15 +1,13 @@
 <?xml version="1.0"?>
 <robot xmlns:xacro="http://www.ros.org/wiki/xacro">
-  <xacro:macro name="panda_arm_sim_ros2_control" params="ns_1 ns_2 hand_1 hand_2 scene_xml mj_yaml">
-    <ros2_control name="FrankaMujocoMultiHardwareInterface" type="system">
+  <xacro:macro name="dual_panda_mjros_ros2_control" params="ns_1 ns_2 hand_1 hand_2">
+    <ros2_control name="FrankaMjHardwareSystem" type="system">
       <hardware>
         <param name="robot_count">2</param>
-        <plugin>franka_hardware/FrankaMujocoMultiHardwareInterface</plugin>
+        <plugin>franka_hardware/FrankaMjHardwareSystem</plugin>
         <param name="ns_1">${ns_1}</param>
         <param name="ns_2">${ns_2}</param>
         <param name="hand_1">${hand_1}</param>
         <param name="hand_2">${hand_2}</param>
-        <param name="scene_xml">${scene_xml}</param>
-        <param name="mj_yaml">${mj_yaml}</param>
       </hardware>
       <xacro:macro name="configure_joint" params="joint_name initial_position">

File: franka_description/robots/sim/dual_panda_arm_sim.urdf.xacro (robot description, xacro)
@@ -5,6 +5,4 @@
   <xacro:arg name="hand_1" default="false"/> <!-- Should a franka_gripper be mounted at the flange?" -->
   <xacro:arg name="hand_2" default="false"/> <!-- Should a franka_gripper be mounted at the flange?" -->
-  <xacro:arg name="scene_xml" default="scene.xml"/> <!-- Path to the scene_xml -->
-  <xacro:arg name="mj_yaml" default=""/> <!-- Path to the scene_xml -->
   <link name="base_link">
     <visual>
@@ -21,5 +19,5 @@
     </collision>
   </link>
-  <xacro:include filename="$(find franka_description)/robots/panda_arm.xacro"/>
+  <xacro:include filename="$(find franka_description)/robots/common/panda_arm.xacro"/>
   <!--
   <xacro:panda_arm arm_id="$(arg arm_id_1)" connected_to="base_link" rpy="${-90 * pi/180} 0 ${-90 * pi/180}"  xyz="-143.26e-3 +600e-3 924.51e-3" safety_distance="0.03"/>
@@ -29,12 +27,12 @@
   <xacro:panda_arm arm_id="$(arg arm_id_2)" connected_to="base_link" rpy="0 0 0"  xyz="0 -0.26 0" safety_distance="0.03"/>
   <xacro:if value="$(arg hand_1)">
-    <xacro:include filename="$(find franka_description)/robots/hand.xacro"/>
+    <xacro:include filename="$(find franka_description)/robots/common/hand.xacro"/>
     <xacro:hand ns="$(arg arm_id_1)" rpy="0 0 ${-pi/4}" connected_to="$(arg arm_id_1)_link8" safety_distance="0.03"/>
   </xacro:if>
   <xacro:if value="$(arg hand_2)">
-    <xacro:include filename="$(find franka_description)/robots/hand.xacro"/>
+    <xacro:include filename="$(find franka_description)/robots/common/hand.xacro"/>
     <xacro:hand ns="$(arg arm_id_2)" rpy="0 0 ${-pi/4}" connected_to="$(arg arm_id_2)_link8" safety_distance="0.03"/>
   </xacro:if>
-  <xacro:include filename="$(find franka_description)/robots/dual_panda_arm_sim.ros2_control.xacro"/>
-  <xacro:panda_arm_sim_ros2_control ns_1="$(arg arm_id_1)" ns_2="$(arg arm_id_2)" hand_1="$(arg hand_1)" hand_2="$(arg hand_2)" scene_xml="$(arg scene_xml)" mj_yaml="$(arg mj_yaml)"/>
+  <xacro:include filename="$(find franka_description)/robots/sim/dual_panda_arm_sim.ros2_control.xacro"/>
+  <xacro:dual_panda_mjros_ros2_control ns_1="$(arg arm_id_1)" ns_2="$(arg arm_id_2)" hand_1="$(arg hand_1)" hand_2="$(arg hand_2)"/>
 </robot>

File: franka_description/robots/sim/panda_arm_sim.ros2_control.xacro (robot description, xacro)
@@ -1,13 +1,11 @@
 <?xml version="1.0"?>
 <robot xmlns:xacro="http://www.ros.org/wiki/xacro">
-  <xacro:macro name="panda_arm_sim_ros2_control" params="ns hand scene_xml mj_yaml">
-    <ros2_control name="FrankaMujocoMultiHardwareInterface" type="system">
+  <xacro:macro name="panda_arm_sim_ros2_control" params="ns hand">
+    <ros2_control name="FrankaMjHardwareSystem" type="system">
       <hardware>
         <param name="robot_count">1</param>
-        <plugin>franka_hardware/FrankaMujocoMultiHardwareInterface</plugin>
+        <plugin>franka_hardware/FrankaMjHardwareSystem</plugin>
         <param name="ns_1">${ns}</param>
         <param name="hand_1">${hand}</param>
-        <param name="scene_xml">${scene_xml}</param>
-        <param name="mj_yaml">${mj_yaml}</param>
       </hardware>
       <xacro:macro name="configure_joint" params="joint_name initial_position">

File: franka_description/robots/sim/panda_arm_sim.urdf.xacro (robot description, xacro)
@@ -3,12 +3,11 @@
   <xacro:arg name="arm_id" default="panda"/> <!-- Name of this panda -->
   <xacro:arg name="hand" default="true"/> <!-- Should a franka_gripper be mounted at the flange?" -->
-  <xacro:arg name="scene_xml" default="scene.xml"/> <!-- Path to the scene_xml -->
-  <xacro:include filename="$(find franka_description)/robots/panda_arm.xacro"/>
+  <xacro:include filename="$(find franka_description)/robots/common/panda_arm.xacro"/>
   <xacro:panda_arm arm_id="$(arg arm_id)" safety_distance="0.03"/>
   <xacro:if value="$(arg hand)">
-    <xacro:include filename="$(find franka_description)/robots/hand.xacro"/>
+    <xacro:include filename="$(find franka_description)/robots/common/hand.xacro"/>
     <xacro:hand ns="$(arg arm_id)" rpy="0 0 ${-pi/4}" connected_to="$(arg arm_id)_link8" safety_distance="0.03"/>
   </xacro:if>
-  <xacro:include filename="$(find franka_description)/robots/panda_arm_mjros.ros2_control.xacro"/>
-  <xacro:panda_arm_sim_ros2_control ns="$(arg arm_id)" hand="$(arg hand)" scene_xml="$(arg scene_xml)"/>
+  <xacro:include filename="$(find franka_description)/robots/sim/panda_arm_sim.ros2_control.xacro"/>
+  <xacro:panda_arm_sim_ros2_control ns="$(arg arm_id)" hand="$(arg hand)"/>
 </robot>
