Commit message: feat: added initial arm position as a parameter in launch

File: franka_description/robots/sim/dual_panda_arm_sim.ros2_control.xacro (robot description, xacro)
@@ -1,5 +1,5 @@
 <?xml version="1.0"?>
 <robot xmlns:xacro="http://www.ros.org/wiki/xacro">
-  <xacro:macro name="dual_panda_mjros_ros2_control" params="ns_1 ns_2 hand_1 hand_2">
+  <xacro:macro name="dual_panda_mjros_ros2_control" params="ns_1 ns_2 hand_1 hand_2 initial_positions_1 initial_positions_2">
     <ros2_control name="FrankaMjHardwareSystem" type="system">
       <hardware>
@@ -22,18 +22,20 @@
         </joint>
       </xacro:macro>
-      <xacro:configure_joint joint_name="${ns_1}_joint1" initial_position="0.0"/>
-      <xacro:configure_joint joint_name="${ns_1}_joint2" initial_position="${-pi/4}"/>
-      <xacro:configure_joint joint_name="${ns_1}_joint3" initial_position="0.0"/>
-      <xacro:configure_joint joint_name="${ns_1}_joint4" initial_position="${-3*pi/4}"/>
-      <xacro:configure_joint joint_name="${ns_1}_joint5" initial_position="0.0"/>
-      <xacro:configure_joint joint_name="${ns_1}_joint6" initial_position="${pi/2}"/>
-      <xacro:configure_joint joint_name="${ns_1}_joint7" initial_position="${pi/4}"/>
-      <xacro:configure_joint joint_name="${ns_2}_joint1" initial_position="0.0"/>
-      <xacro:configure_joint joint_name="${ns_2}_joint2" initial_position="${-pi/4}"/>
-      <xacro:configure_joint joint_name="${ns_2}_joint3" initial_position="0.0"/>
-      <xacro:configure_joint joint_name="${ns_2}_joint4" initial_position="${-3*pi/4}"/>
-      <xacro:configure_joint joint_name="${ns_2}_joint5" initial_position="0.0"/>
-      <xacro:configure_joint joint_name="${ns_2}_joint6" initial_position="${pi/2}"/>
-      <xacro:configure_joint joint_name="${ns_2}_joint7" initial_position="${pi/4}"/>
+      <xacro:property name="initial_positions_list_1" value="${initial_positions_1.split(' ')}"/>
+      <xacro:property name="initial_positions_list_2" value="${initial_positions_2.split(' ')}"/>
+      <xacro:configure_joint joint_name="${ns_1}_joint1" initial_position="${initial_positions_list_1[0]}"/>
+      <xacro:configure_joint joint_name="${ns_1}_joint2" initial_position="${initial_positions_list_1[1]}"/>
+      <xacro:configure_joint joint_name="${ns_1}_joint3" initial_position="${initial_positions_list_1[2]}"/>
+      <xacro:configure_joint joint_name="${ns_1}_joint4" initial_position="${initial_positions_list_1[3]}"/>
+      <xacro:configure_joint joint_name="${ns_1}_joint5" initial_position="${initial_positions_list_1[4]}"/>
+      <xacro:configure_joint joint_name="${ns_1}_joint6" initial_position="${initial_positions_list_1[5]}"/>
+      <xacro:configure_joint joint_name="${ns_1}_joint7" initial_position="${initial_positions_list_1[6]}"/>
+      <xacro:configure_joint joint_name="${ns_2}_joint1" initial_position="${initial_positions_list_2[0]}"/>
+      <xacro:configure_joint joint_name="${ns_2}_joint2" initial_position="${initial_positions_list_2[1]}"/>
+      <xacro:configure_joint joint_name="${ns_2}_joint3" initial_position="${initial_positions_list_2[2]}"/>
+      <xacro:configure_joint joint_name="${ns_2}_joint4" initial_position="${initial_positions_list_2[3]}"/>
+      <xacro:configure_joint joint_name="${ns_2}_joint5" initial_position="${initial_positions_list_2[4]}"/>
+      <xacro:configure_joint joint_name="${ns_2}_joint6" initial_position="${initial_positions_list_2[5]}"/>
+      <xacro:configure_joint joint_name="${ns_2}_joint7" initial_position="${initial_positions_list_2[6]}"/>
     </ros2_control>
   </xacro:macro>

File: franka_description/robots/sim/dual_panda_arm_sim.urdf.xacro (robot description, xacro)
@@ -5,4 +5,6 @@
   <xacro:arg name="hand_1" default="false"/> <!-- Should a franka_gripper be mounted at the flange?" -->
   <xacro:arg name="hand_2" default="false"/> <!-- Should a franka_gripper be mounted at the flange?" -->
+  <xacro:arg name="initial_positions_1" default="0.0 ${-pi/4} 0.0 ${-3*pi/4} 0.0 ${pi/2} ${pi/4}"/> <!-- initial joint positions of the robot-->
+  <xacro:arg name="initial_positions_2" default="0.0 ${-pi/4} 0.0 ${-3*pi/4} 0.0 ${pi/2} ${pi/4}"/> <!-- initial joint positions of the robot-->
   <link name="base_link">
     <visual>
@@ -35,4 +37,10 @@
   </xacro:if>
   <xacro:include filename="$(find franka_description)/robots/sim/dual_panda_arm_sim.ros2_control.xacro"/>
-  <xacro:dual_panda_mjros_ros2_control ns_1="$(arg arm_id_1)" ns_2="$(arg arm_id_2)" hand_1="$(arg hand_1)" hand_2="$(arg hand_2)"/>
+  <xacro:dual_panda_mjros_ros2_control
+      ns_1="$(arg arm_id_1)"
+      ns_2="$(arg arm_id_2)"
+      hand_1="$(arg hand_1)"
+      hand_2="$(arg hand_2)"
+      initial_positions_1="$(arg initial_positions_1)"
+      initial_positions_2="$(arg initial_positions_2)"/>
 </robot>

File: franka_description/robots/sim/panda_arm_sim.ros2_control.xacro (robot description, xacro)
@@ -1,5 +1,5 @@
 <?xml version="1.0"?>
 <robot xmlns:xacro="http://www.ros.org/wiki/xacro">
-  <xacro:macro name="panda_arm_sim_ros2_control" params="ns hand">
+  <xacro:macro name="panda_arm_sim_ros2_control" params="ns hand initial_positions">
     <ros2_control name="FrankaMjHardwareSystem" type="system">
       <hardware>
@@ -20,11 +20,12 @@
         </joint>
       </xacro:macro>
-      <xacro:configure_joint joint_name="${ns}_joint1" initial_position="0.0"/>
-      <xacro:configure_joint joint_name="${ns}_joint2" initial_position="${-pi/4}"/>
-      <xacro:configure_joint joint_name="${ns}_joint3" initial_position="0.0"/>
-      <xacro:configure_joint joint_name="${ns}_joint4" initial_position="${-3*pi/4}"/>
-      <xacro:configure_joint joint_name="${ns}_joint5" initial_position="0.0"/>
-      <xacro:configure_joint joint_name="${ns}_joint6" initial_position="${pi/2}"/>
-      <xacro:configure_joint joint_name="${ns}_joint7" initial_position="${pi/4}"/>
+      <xacro:property name="initial_positions_list" value="${initial_positions.split(' ')}"/>
+      <xacro:configure_joint joint_name="${ns}_joint1" initial_position="${initial_positions_list[0]}"/>
+      <xacro:configure_joint joint_name="${ns}_joint2" initial_position="${initial_positions_list[1]}"/>
+      <xacro:configure_joint joint_name="${ns}_joint3" initial_position="${initial_positions_list[2]}"/>
+      <xacro:configure_joint joint_name="${ns}_joint4" initial_position="${initial_positions_list[3]}"/>
+      <xacro:configure_joint joint_name="${ns}_joint5" initial_position="${initial_positions_list[4]}"/>
+      <xacro:configure_joint joint_name="${ns}_joint6" initial_position="${initial_positions_list[5]}"/>
+      <xacro:configure_joint joint_name="${ns}_joint7" initial_position="${initial_positions_list[6]}"/>
     </ros2_control>
   </xacro:macro>

File: franka_description/robots/sim/panda_arm_sim.urdf.xacro (robot description, xacro)
@@ -3,4 +3,5 @@
   <xacro:arg name="arm_id" default="panda"/> <!-- Name of this panda -->
   <xacro:arg name="hand" default="true"/> <!-- Should a franka_gripper be mounted at the flange?" -->
+  <xacro:arg name="initial_positions" default="0.0 ${-pi/4} 0.0 ${-3*pi/4} 0.0 ${pi/2} ${pi/4}"/> <!-- initial joint positions of the robot-->
   <xacro:include filename="$(find franka_description)/robots/common/panda_arm.xacro"/>
   <xacro:panda_arm arm_id="$(arg arm_id)" safety_distance="0.03"/>
@@ -10,4 +11,4 @@
   </xacro:if>
   <xacro:include filename="$(find franka_description)/robots/sim/panda_arm_sim.ros2_control.xacro"/>
-  <xacro:panda_arm_sim_ros2_control ns="$(arg arm_id)" hand="$(arg hand)"/>
+  <xacro:panda_arm_sim_ros2_control ns="$(arg arm_id)" hand="$(arg hand)" initial_positions="$(arg initial_positions)"/>
 </robot>
