Commit message: chg: reorganize garmi-specific description files

File: garmi_packages/garmi_description/robots/base.xacro (robot description, xacro)
@@ -16,5 +16,5 @@
       <visual>
         <geometry>
-          <mesh filename="package://franka_description/meshes/visual/torso.dae" scale="1 1 1"/>
+          <mesh filename="package://garmi_description/robot/meshes/torso.dae" scale="1 1 1"/>
         </geometry>
       </visual>

File: garmi_packages/garmi_description/robots/head.xacro (robot description, xacro)
@@ -27,5 +27,5 @@
         <origin xyz="0 0 0" rpy="0 0 0" />
         <geometry>
-          <mesh filename="package://franka_description/meshes/visual/head.dae" scale="1 1 1"/>
+          <mesh filename="package://garmi_description/robots/meshes/head.dae" scale="1 1 1"/>
         </geometry>
       </visual>

File: garmi_packages/garmi_description/robots/lidar_with_wheel_mount.xacro (robot description, xacro)
@@ -1,5 +1,5 @@
 <?xml version="1.0"?>
 <robot xmlns:xacro="http://www.ros.org/wiki/xacro" >
-  <xacro:include filename="$(find franka_description)/sensors/rplidarA2.xacro" />
+  <xacro:include filename="$(find garmi_description)/robots/rplidarA2.xacro" />
   <xacro:macro name="lidar" params="connected_to ns:='lidar' xyz:='0 0 0' rpy:='0 0 0' ">
     <link name="${ns}_mount" >

File: garmi_packages/garmi_description/robots/mobile_platform.xacro (robot description, xacro)
@@ -11,5 +11,5 @@
       <visual>
         <geometry>
-          <mesh filename="package://franka_description/meshes/visual/mobile_platform.dae" scale="1 1 1"/>
+          <mesh filename="package://garmi_description/robots/meshes/mobile_platform.dae" scale="1 1 1"/>
         </geometry>
         <origin rpy="0 0 ${+90 * pi/180}" xyz="0 0 -0.21"/>

File: garmi_packages/garmi_description/robots/rplidarA2.xacro (robot description, xacro)
@@ -42,5 +42,5 @@
       <visual>
         <geometry>
-          <mesh filename="package://garmi_robot_description/meshes/visual/rplidarA2.dae" />
+          <mesh filename="package://garmi_description/robots/meshes/rplidarA2.dae" />
         </geometry>
       </visual>

Commit message: feat: add lidar to garmi description

File: garmi_packages/garmi_description/robots/base.xacro (robot description, xacro)
@@ -16,5 +16,5 @@
       <visual>
         <geometry>
-          <mesh filename="package://garmi_description/robot/meshes/torso.dae" scale="1 1 1"/>
+          <mesh filename="package://garmi_description/robots/meshes/torso.dae" scale="1 1 1"/>
         </geometry>
       </visual>

File: garmi_packages/garmi_description/robots/garmi_sim.urdf.xacro (robot description, xacro)
@@ -13,5 +13,5 @@
   <xacro:include filename="$(find garmi_description)/robots/garmi_wheel.xacro" />
   <xacro:include filename="$(find garmi_description)/robots/mobile_platform.xacro" />
-  <!-- <xacro:include filename="$(find franka_description)/robots/lidar_with_wheel_mount.xacro" /> -->
+  <xacro:include filename="$(find garmi_description)/robots/lidar_with_wheel_mount.xacro" />
   <link name="base_link" />
   <!-- left arm with gripper -->
@@ -32,6 +32,6 @@
   <xacro:garmi_wheel wheel_id="left" connected_to="base_link" rpy="${-90 * pi/180} 0 0" xyz="0 0.375 -0.125" />
   <xacro:garmi_wheel wheel_id="right" connected_to="base_link" rpy="${90 * pi/180} 0 0" xyz="0 -0.375 -0.125" />
-  <!-- <xacro:lidar connected_to="base_link" xyz="0.42 0 0" rpy="0 0 ${pi}" ns="lidar_front" />
-  <xacro:lidar connected_to="base_link" xyz="-0.42 0 0" rpy="0 0 0.05" ns="lidar_rear" /> -->
+  <xacro:lidar connected_to="base_link" xyz="0.42 0 0.01" rpy="0 0 ${pi}" ns="lidar_front" />
+  <xacro:lidar connected_to="base_link" xyz="-0.42 0 0.01" rpy="0 0 0.05" ns="lidar_rear" />
   <xacro:include filename="$(find franka_description)/robots/sim/dual_panda_arm_sim.ros2_control.xacro"/>
   <xacro:dual_panda_mjros_ros2_control  ns_1="$(arg arm_id_1)"

File: garmi_packages/garmi_description/robots/lidar_with_wheel_mount.xacro (robot description, xacro)
@@ -1,5 +1,5 @@
 <?xml version="1.0"?>
 <robot xmlns:xacro="http://www.ros.org/wiki/xacro" >
-  <xacro:include filename="$(find garmi_description)/robots/rplidarA2.xacro" />
+  <xacro:include filename="$(find garmi_description)/robots/rplidarA2_kinematics.xacro" />
   <xacro:macro name="lidar" params="connected_to ns:='lidar' xyz:='0 0 0' rpy:='0 0 0' ">
     <link name="${ns}_mount" >
@@ -14,5 +14,5 @@
         <origin xyz="0 0 0" rpy="0 0 0" />
         <geometry>
-           <box size="0.1 0.1 0.1" />
+           <box size="0.01 0.01 0.01" />
         </geometry>
       </visual>
