Commit message: clean the code, remove useless code

File: franka_description/robots/common/metal_ball.xacro (robot description, xacro)
@@ -1,5 +1,5 @@
 <?xml version='1.0' encoding='utf-8'?>
 <robot xmlns:xacro="http://www.ros.org/wiki/xacro">
-  <xacro:macro name="metal_ball" params="ns connected_to radius:=0.03 mass:=0.2 xyz:='0 0 0.03' tcp_xyz:='0 0 0.06' rgba:='0.72 0.74 0.76 1.0'">
+  <xacro:macro name="metal_ball" params="ns connected_to radius:=0.03 mass:=0.2 xyz:='0 0 0.03' rgba:='0.72 0.74 0.76 1.0'">
     <link name="${ns}_metal_ball_link">
       <visual>
@@ -34,5 +34,5 @@
     <link name="${ns}_metal_ball_tcp_link"/>
     <joint name="${ns}_metal_ball_tcp_joint" type="fixed">
-      <origin xyz="${tcp_xyz}" rpy="0 0 0"/>
+      <origin xyz="${xyz}" rpy="0 0 0"/>
       <parent link="${connected_to}"/>
       <child link="${ns}_metal_ball_tcp_link"/>

File: franka_description/robots/real/panda_arm.urdf.xacro (robot description, xacro)
@@ -10,5 +10,4 @@
   <xacro:arg name="metal_ball_mass" default="0.2"/>
   <xacro:arg name="metal_ball_xyz" default="0 0 0.03"/>
-  <xacro:arg name="metal_ball_tcp_xyz" default="0 0 0.06"/>
   <xacro:include filename="$(find franka_description)/robots/common/panda_arm.xacro"/>
   <xacro:panda_arm arm_id="$(arg arm_id)" safety_distance="0.03"/>
@@ -24,6 +23,5 @@
       radius="$(arg metal_ball_radius)"
       mass="$(arg metal_ball_mass)"
-      xyz="$(arg metal_ball_xyz)"
-      tcp_xyz="$(arg metal_ball_tcp_xyz)"/>
+      xyz="$(arg metal_ball_xyz)"/>
   </xacro:if>
   <xacro:include filename="$(find franka_description)/robots/real/panda_arm.ros2_control.xacro"/>

File: franka_description/robots/sim/panda_arm_sim.urdf.xacro (robot description, xacro)
@@ -8,5 +8,4 @@
   <xacro:arg name="metal_ball_mass" default="0.2"/>
   <xacro:arg name="metal_ball_xyz" default="0 0 0.03"/>
-  <xacro:arg name="metal_ball_tcp_xyz" default="0 0 0.06"/>
   <xacro:include filename="$(find franka_description)/robots/common/panda_arm.xacro"/>
   <xacro:panda_arm arm_id="$(arg arm_id)" safety_distance="0.03"/>
@@ -22,6 +21,5 @@
       radius="$(arg metal_ball_radius)"
       mass="$(arg metal_ball_mass)"
-      xyz="$(arg metal_ball_xyz)"
-      tcp_xyz="$(arg metal_ball_tcp_xyz)"/>
+      xyz="$(arg metal_ball_xyz)"/>
   </xacro:if>
   <xacro:include filename="$(find franka_description)/robots/sim/panda_arm_sim.ros2_control.xacro"/>
