Commit message: feat: working moveit configuration for two pandas

File: franka_moveit_config/srdf/dual_panda.srdf.xacro (robot description, xacro)
@@ -5,32 +5,38 @@
   <xacro:arg name="hand_1" default="false"/>
   <xacro:arg name="hand_2" default="false"/>
-  <!-- <xacro:arg name="hand_group_1" default="left_hand"/> -->
-  <!-- <xacro:arg name="hand_group_2" default="right_hand"/> -->
   <xacro:arg name="parent_frame" default="world"/>
   <xacro:property name="arm_id_1" value="$(arg arm_id_1)"/>
   <xacro:property name="arm_id_2" value="$(arg arm_id_2)"/>
-  <!-- <xacro:property name="hand_group_1" value="$(arg hand_group_1)"/> -->
-  <!-- <xacro:property name="hand_group_2" value="$(arg hand_group_2)"/> -->
   <xacro:include filename="$(find franka_moveit_config)/srdf/dual_panda_arm.xacro"/>
   <xacro:dual_panda_arm arm_id="${arm_id_1}" />
   <xacro:dual_panda_arm arm_id="${arm_id_2}" />
   <virtual_joint name="virtual_joint" type="fixed" parent_frame="$(arg parent_frame)" child_link="base_link"/>
-  <!-- <xacro:arm_groups side="${arm_id_1}"/> -->
-  <!-- <xacro:arm_groups side="${arm_id_2}"/> -->
   <group name="dual_panda">
     <group name="${arm_id_1}_arm"/>
     <group name="${arm_id_2}_arm"/>
+    <xacro:if value="$(arg hand_1)">
+      <group name="${arm_id_1}_manipulator"/>
+    </xacro:if>
+    <xacro:if value="$(arg hand_2)">
+      <group name="${arm_id_2}_manipulator"/>
+    </xacro:if>
   </group>
-  <!-- <xacro:if value="$(arg hand_1)">
-    <xacro:include filename="$(find franka_moveit_config)/srdf/hand.xacro"/>
-    <xacro:hand arm_id="${arm_id_1}" group_name="${arm_id_1}_arm"/>
-    <xacro:include filename="$(find franka_moveit_config)/srdf/panda_arm_hand.xacro"/>
-    <xacro:panda_arm_hand arm_id="${arm_id_1}" group_name="${arm_id_1}_arm"/>
+  <xacro:include filename="$(find franka_moveit_config)/srdf/dual_group_definition.xacro"/>
+  <xacro:if value="$(arg hand_1)">
+    <!-- <xacro:group_definition arm_id="${arm_id_1}" group_name="${arm_id_1}_arm" tip_link="${arm_id_1}_link8"/> -->
+    <xacro:group_definition arm_id="${arm_id_1}" group_name="${arm_id_1}_manipulator" tip_link="${arm_id_1}_hand_tcp"/>
+    <xacro:include filename="$(find franka_moveit_config)/srdf/dual_hand.xacro"/>
+    <xacro:hand arm_id="${arm_id_1}"/>
+    <xacro:include filename="$(find franka_moveit_config)/srdf/dual_panda_arm_hand.xacro"/>
+    <xacro:panda_arm_hand arm_id="${arm_id_1}"/>
   </xacro:if>
+<!--  -->
   <xacro:if value="$(arg hand_2)">
-    <xacro:include filename="$(find franka_moveit_config)/srdf/hand.xacro"/>
-    <xacro:hand arm_id="${arm_id_2}" group_name="${arm_id_1}_arm"/>
-    <xacro:include filename="$(find franka_moveit_config)/srdf/panda_arm_hand.xacro"/>
-    <xacro:panda_arm_hand arm_id="${arm_id_2}" group_name="${arm_id_1}_arm"/>
-  </xacro:if> -->
+    <!-- <xacro:group_definition arm_id="${arm_id_2}" group_name="${arm_id_2}_arm" tip_link="${arm_id_2}_link8"/> -->
+    <xacro:group_definition arm_id="${arm_id_2}" group_name="${arm_id_2}_manipulator" tip_link="${arm_id_2}_hand_tcp"/>
+    <xacro:include filename="$(find franka_moveit_config)/srdf/dual_hand.xacro"/>
+    <xacro:hand arm_id="${arm_id_2}"/>
+    <xacro:include filename="$(find franka_moveit_config)/srdf/dual_panda_arm_hand.xacro"/>
+    <xacro:panda_arm_hand arm_id="${arm_id_2}"/>
+  </xacro:if>
 </robot>

File: franka_moveit_config/srdf/dual_panda_arm.xacro (robot description, xacro)
@@ -2,7 +2,9 @@
 <robot xmlns:xacro="http://www.ros.org/wiki/xacro" name="dual_panda">
   <xacro:macro name="dual_panda_arm" params="arm_id='panda'">
-    <group name="${arm_id}_arm">
+    <xacro:include filename="$(find franka_moveit_config)/srdf/dual_group_definition.xacro"/>
+    <xacro:group_definition arm_id="${arm_id}" group_name="${arm_id}_arm" tip_link="${arm_id}_link8"/>
+    <!-- <group name="${arm_id}_arm">
       <chain base_link="${arm_id}_link0" tip_link="${arm_id}_link8" />
-    </group>
+    </group> -->
     <disable_collisions link1="${arm_id}_link0" link2="${arm_id}_link1" reason="Adjacent" />
     <disable_collisions link1="${arm_id}_link0" link2="${arm_id}_link2" reason="Never" />
