Commit message: nonlinear control  inertial result not good

File: model_urdf/panda_ng.urdf (robot description, URDF)
Before this commit: robot panda, 9 links, 8 joints
Links:
- link panda_link0: mass None -> 0.629769
- link panda_link1: mass None -> 4.970684
- link panda_link2: mass None -> 0.646926
- link panda_link3: mass None -> 3.228604
- link panda_link4: mass None -> 3.587895
- link panda_link5: mass None -> 1.225946
- link panda_link6: mass None -> 1.666555
- link panda_link7: mass None -> 0.735522
